File: PCB/ClockCubed_v1.sch (EAGLE design)
At the start: 107 parts, among them IC1 74LS595D, IC10 A1321LH, IC11 A1321LH, IC12 A1321LH, IC2 74LS595D, IC3 74LS595D, IC4 74LS595D, IC5 74LS595D, IC6 74LS595D, IC7 74LS595D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

Commit message: updated license, added pdf files of board and sch
updated names in license, created pdf files of schematic and layout
files, added copyright to schematic
Other:
- note added: "All Rights Reserved"
- note added: "Clock Cubed V1"
- note added: "Copyright (c) 2014, Kevin Baker and Lucas Lappe"
- note added: "Licensed under BSD"
- note added: "PNP, not NPN"
Changed lines of the file:
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@@
 <?xml version="1.0" encoding="utf-8"?>
 <!DOCTYPE eagle SYSTEM "eagle.dtd">
-<eagle version="6.1">
+<eagle version="6.5.0">
 <drawing>
 <settings>
@@
 <text x="149.86" y="294.894" size="1.778" layer="97">UVLO 2.6V</text>
 <text x="131.572" y="317.754" size="1.778" layer="97">*close jumper SJ2 to disable UVLO*</text>
+<text x="297.18" y="304.8" size="3.81" layer="91">Clock Cubed V1</text>
+<text x="297.18" y="297.18" size="3.81" layer="91">Copyright (c) 2014, Kevin Baker and Lucas Lappe</text>
+<text x="297.18" y="289.56" size="3.81" layer="91">All Rights Reserved</text>
+<text x="297.18" y="281.94" size="3.81" layer="91">Licensed under BSD</text>
+<text x="236.22" y="-50.8" size="3.81" layer="91">PNP, not NPN</text>
+<text x="345.44" y="-53.34" size="3.81" layer="91">PNP, not NPN</text>
 </plain>
 <instances>
